File: PCB BLINK/PCB BLINK.kicad_sch (KiCad schematic)
At the start: 5 parts, among them U2 HC-SR04, U3 ER_OLEDM0.91_1x-I2C

Commit message: case and pcb production
Parts:
- removed U3: ER_OLEDM0.91_1x-I2C, Display:ER_OLEDM0.91_1x-I2C, symbol Display_Graphic:ER_OLEDM0.91_1x-I2C
- added Brd1: SSD1306, SSD1306:128x64OLED, symbol SSD1306 OLED 0.96{dblquote}:SSD1306
Connections:
- net GND: now also Brd1.1 (GND)
- net at U1.16 (3.3v): now also Brd1.2 (VCC)
- net at U1.26 (GPIO21): now also Brd1.4 (SDA)
- net at U1.29 (GPIO22): now also Brd1.3 (SCL)
Changed lines of the file:
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@@
 	(paper "A4")
 	(junction
-		(at 130.81 101.6)
+		(at 137.16 111.76)
 		(diameter 0)
 		(color 0 0 0 0)
@@
 	(wire
 		(pts
-			(xy 140.97 109.22) (xy 149.86 109.22)
+			(xy 149.86 83.82) (xy 146.05 83.82)
 		)
 		(stroke
@@
 	(wire
 		(pts
+			(xy 146.05 83.82) (xy 146.05 114.3)
+		)
+		(stroke
+			(width 0)
+			(type default)
+		)
+	)
+	(wire
+		(pts
+			(xy 146.05 114.3) (xy 137.16 114.3)
+		)
+		(stroke
+			(width 0)
+			(type default)
+		)
+	)
+	(wire
+		(pts
 			(xy 142.24 101.6) (xy 149.86 101.6)
 		)
@@
 	(wire
 		(pts
-			(xy 147.32 83.82) (xy 149.86 83.82)
-		)
-		(stroke
-			(width 0)
-			(type default)
-		)
-	)
-	(wire
-		(pts
-			(xy 118.11 93.98) (xy 147.32 93.98)
-		)
-		(stroke
-			(width 0)
-			(type default)
-		)
-	)
-	(wire
-		(pts
 			(xy 142.24 88.9) (xy 142.24 101.6)
 		)
@@
 	(wire
 		(pts
-			(xy 140.97 114.3) (xy 140.97 116.84)
+			(xy 137.16 109.22) (xy 137.16 111.76)
 		)
 		(stroke
@@
 	(wire
 		(pts
-			(xy 147.32 93.98) (xy 147.32 83.82)
-		)
-		(stroke
-			(width 0)
-			(type default)
-		)
-	)
-	(wire
-		(pts
-			(xy 140.97 116.84) (xy 149.86 116.84)
+			(xy 137.16 116.84) (xy 149.86 116.84)
 		)
 		(stroke
@@
 	(wire
 		(pts
-			(xy 118.11 124.46) (xy 118.11 93.98)
-		)
-		(stroke
-			(width 0)
-			(type default)
-		)
-	)
-	(wire
-		(pts
 			(xy 133.35 88.9) (xy 142.24 88.9)
 		)
@@
 	(wire
 		(pts
+			(xy 147.32 109.22) (xy 147.32 119.38)
+		)
+		(stroke
+			(width 0)
+			(type default)
+		)
+	)
+	(wire
+		(pts
+			(xy 149.86 109.22) (xy 147.32 109.22)
+		)
+		(stroke
+			(width 0)
+			(type default)
+		)
+	)
+	(wire
+		(pts
+			(xy 147.32 119.38) (xy 137.16 119.38)
+		)
+		(stroke
+			(width 0)
+			(type default)
+		)
+	)
+	(wire
+		(pts
 			(xy 115.57 86.36) (xy 115.57 81.28)
 		)
@@
 			(type default)
 			(color 0 0 0 1)
-		)
-	)
-	(wire
-		(pts
-			(xy 123.19 101.6) (xy 130.81 101.6)
-		)
-		(stroke
-			(width 0)
-			(type default)
-		)
-	)
-	(wire
-		(pts
-			(xy 130.81 121.92) (xy 130.81 124.46)
-		)
-		(stroke
-			(width 0)
-			(type default)
-		)
-	)
-	(wire
-		(pts
-			(xy 130.81 124.46) (xy 118.11 124.46)
-		)
-		(stroke
-			(width 0)
-			(type default)
 		)
 	)
@@
 				(path "/045d4c76-b8e6-4e35-9741-edeedb73b92f"
 					(reference "R1")
+					(unit 1)
+				)
+			)
+		)
+	)
+	(symbol
+		(lib_id "SSD1306 OLED 0.96{dblquote}:SSD1306")
+		(at 128.27 115.57 270)
+		(unit 1)
+		(body_style 1)
+		(exclude_from_sim no)
+		(in_bom yes)
+		(on_board yes)
+		(in_pos_files yes)
+		(dnp no)
+		(fields_autoplaced yes)
+		(property "Reference" "Brd1"
+			(at 128.27 104.14 90)
+			(hide yes)
+			(show_name no)
+			(do_not_autoplace no)
+			(effects
+				(font
+					(size 1.27 1.27)
+				)
+			)
+		)
+		(property "Value" "SSD1306"
+			(at 128.27 106.68 90)
+			(hide yes)
+			(show_name no)
+			(do_not_autoplace no)
+			(effects
+				(font
+					(size 1.27 1.27)
+				)
+			)
+		)
+		(property "Footprint" "SSD1306:128x64OLED"
+			(at 134.62 115.57 0)
+			(hide yes)
+			(show_name no)
+			(do_not_autoplace no)
+			(effects
+				(font
+					(size 1.27 1.27)
+				)
+			)
+		)
+		(property "Datasheet" ""
+			(at 134.62 115.57 0)
+			(hide yes)
+			(show_name no)
+			(do_not_autoplace no)
+			(effects
+				(font
+					(size 1.27 1.27)
+				)
+			)
+		)
+		(property "Description" "SSD1306 OLED"
+			(at 128.27 115.57 0)
+			(hide yes)
+			(show_name no)
+			(do_not_autoplace no)
+			(effects
+				(font
+					(size 1.27 1.27)
+				)
+			)
+		)
+		(pin "4"
+		)
+		(pin "1"
+		)
+		(pin "2"
+		)
+		(pin "3"
+		)
+		(instances
+			(project "PCB BLINK"
+				(path "/045d4c76-b8e6-4e35-9741-edeedb73b92f"
+					(reference "Brd1")
 					(unit 1)
 				)
@@
 	(symbol
 		(lib_id "power:GND")
-		(at 130.81 101.6 180)
+		(at 137.16 111.76 90)
 		(unit 1)
 		(body_style 1)
@@
 		(dnp no)
 		(fields_autoplaced yes)
-		(property "Reference" "#PWR02"
-			(at 130.81 95.25 0)
+		(property "Reference" "#PWR01"
+			(at 143.51 111.76 0)
 			(hide yes)
 			(show_name no)
@@
 		)
 		(property "Value" "GND"
-			(at 130.81 96.52 0)
-			(show_name no)
-			(do_not_autoplace no)
-			(effects
-				(font
-					(size 1.27 1.27)
-				)
+			(at 140.97 111.7599 90)
+			(show_name no)
+			(do_not_autoplace no)
+			(effects
+				(font
+					(size 1.27 1.27)
+				)
+				(justify right)
 			)
 		)
 		(property "Footprint" ""
-			(at 130.81 101.6 0)
+			(at 137.16 111.76 0)
 			(hide yes)
 			(show_name no)
@@
 		)
 		(property "Datasheet" ""
-			(at 130.81 101.6 0)
+			(at 137.16 111.76 0)
 			(hide yes)
 			(show_name no)
@@
 		)
 		(property "Description" "Power symbol creates a global label with name \"GND\" , ground"
-			(at 130.81 101.6 0)
+			(at 137.16 111.76 0)
 			(hide yes)
 			(show_name no)
@@
 			(project "PCB BLINK"
 				(path "/045d4c76-b8e6-4e35-9741-edeedb73b92f"
-					(reference "#PWR02")
+					(reference "#PWR01")
 					(unit 1)
 				)
@@
 	(symbol
 		(lib_id "power:PWR_FLAG")
-		(at 123.19 101.6 0)
+		(at 137.16 109.22 0)
 		(unit 1)
 		(body_style 1)
@@
 		(dnp no)
 		(property "Reference" "#FLG01"
-			(at 123.19 99.695 0)
+			(at 137.16 107.315 0)
 			(hide yes)
 			(show_name no)
@@
 		)
 		(property "Value" "PWR_FLAG"
-			(at 123.19 97.79 0)
-			(show_name no)
-			(do_not_autoplace no)
-			(effects
-				(font
-					(size 1.27 1.27)
-				)
+			(at 132.842 104.902 0)
+			(show_name no)
+			(do_not_autoplace no)
+			(effects
+				(font
+					(size 1.27 1.27)
+				)
+				(justify left)
 			)
 		)
 		(property "Footprint" ""
-			(at 123.19 101.6 0)
+			(at 137.16 109.22 0)
 			(hide yes)
 			(show_name no)
@@
 		)
 		(property "Datasheet" ""
-			(at 123.19 101.6 0)
+			(at 137.16 109.22 0)
 			(hide yes)
 			(show_name no)
@@
 		)
 		(property "Description" "Special symbol for telling ERC where power comes from"
-			(at 123.19 101.6 0)
+			(at 137.16 109.22 0)
 			(hide yes)
 			(show_name no)
@@
 				(path "/045d4c76-b8e6-4e35-9741-edeedb73b92f"
 					(reference "#FLG01")
-					(unit 1)
-				)
-			)
-		)
-	)
-	(symbol
-		(lib_id "Display_Graphic:ER_OLEDM0.91_1x-I2C")
-		(at 130.81 111.76 180)
-		(unit 1)
-		(body_style 1)
-		(exclude_from_sim no)
-		(in_bom yes)
-		(on_board yes)
-		(in_pos_files yes)
-		(dnp no)
-		(property "Reference" "U3"
-			(at 118.11 111.76 90)
-			(show_name no)
-			(do_not_autoplace no)
-			(effects
-				(font
-					(size 1.27 1.27)
-				)
-				(justify left)
-			)
-		)
-		(property "Value" "ER_OLEDM0.91_1x-I2C"
-			(at 120.65 101.6 90)
-			(show_name no)
-			(do_not_autoplace no)
-			(effects
-				(font
-					(size 1.27 1.27)
-				)
-				(justify left)
-			)
-		)
-		(property "Footprint" "Display:ER_OLEDM0.91_1x-I2C"
-			(at 112.776 99.06 0)
-			(hide yes)
-			(show_name no)
-			(do_not_autoplace no)
-			(effects
-				(font
-					(size 1.27 1.27)
-				)
-			)
-		)
-		(property "Datasheet" "https://www.buydisplay.com/download/manual/ER-OLEDM0.91-1_Datasheet.pdf"
-			(at 88.138 97.028 0)
-			(hide yes)
-			(show_name no)
-			(do_not_autoplace no)
-			(effects
-				(font
-					(size 1.27 1.27)
-				)
-			)
-		)
-		(property "Description" "SSD1306 OLED module, 0.91 inch, 128x32, I2C"
-			(at 104.14 94.996 0)
-			(hide yes)
-			(show_name no)
-			(do_not_autoplace no)
-			(effects
-				(font
-					(size 1.27 1.27)
-				)
-			)
-		)
-		(pin "1"
-		)
-		(pin "3"
-		)
-		(pin "2"
-		)
-		(pin "4"
-		)
-		(instances
-			(project "PCB BLINK"
-				(path "/045d4c76-b8e6-4e35-9741-edeedb73b92f"
-					(reference "U3")
 					(unit 1)
 				)
@@
 		)
 	)
-	(group ""
-		(members "016ed10b-db4f-4a33-960d-d7ae80886bfe" "09212be4-ba44-488b-8277-c5c9fee62019")
-	)
-	(group ""
-		(members "091d2677-27d5-42a3-9b64-099f62908d97" "8aa91f1f-615c-4e3d-a753-3d08cd6267c2")
-	)
 	(sheet_instances
